File: karca_v2/curr_monitor.kicad_sch (KiCad schematic)
At the start: 31 parts, among them U28 MCP3204, U29 INA180A4

Commit message: Version alpha
Parts:
- removed C71: 0.1u, symbol Device:C
- removed D21, D22, D4, D6, D7: D_Schottky, Diode_SMD:D_SMA, symbol Device:D_Schottky
- removed unit 2 of U27
- removed unit 3 of U27
- removed U28: MCP3204, symbol Analog_ADC:MCP3204
- added unit 3 of U31
- added unit 2 of U31
- added U32: NUP4202, Package_SO:TSOP-6_1.65x3.05mm_P0.95mm, symbol Power_Protection:NUP4202
- C51: renamed from C63; footprint (none) -> Capacitor_SMD:C_1206_3216Metric
- C52: renamed from C64; value 68n -> 0.1u
- C54: renamed from C67; value 68n -> 0.1u
- C55: renamed from C69; value 68n -> 0.1u
- C56: renamed from C65; footprint (none) -> Capacitor_SMD:C_0402_1005Metric
- C57: renamed from C68; value 68n -> 0.1u
- C58: renamed from C70; value 68n -> 0.1u
- R100: renamed from R30; footprint (none) -> Resistor_SMD:R_1206_3216Metric
- R101: renamed from R100; value 910 -> 1k; footprint (none) -> Resistor_SMD:R_1206_3216Metric
- R102: renamed from R31; footprint (none) -> Resistor_SMD:R_1206_3216Metric
- R103: renamed from R104; value 910 -> 1k; footprint (none) -> Resistor_SMD:R_1206_3216Metric
- R104: renamed from R32; footprint (none) -> Resistor_SMD:R_1206_3216Metric
- R105: renamed from R103; value 910 -> 1k; footprint (none) -> Resistor_SMD:R_1206_3216Metric
- R106: renamed from R33; footprint (none) -> Resistor_SMD:R_1206_3216Metric
- R107: renamed from R105; value 910 -> 1k; footprint (none) -> Resistor_SMD:R_1206_3216Metric
- R98: renamed from R35; footprint (none) -> Resistor_SMD:R_1206_3216Metric
- R99: renamed from R55; value 910 -> 1k; footprint (none) -> Resistor_SMD:R_1206_3216Metric
- TP55: renamed from TP4; footprint (none) -> TestPoint:TestPoint_Pad_D2.0mm
- TP56: renamed from TP46; footprint (none) -> TestPoint:TestPoint_Pad_D2.0mm
- TP57: renamed from TP48; footprint (none) -> TestPoint:TestPoint_Pad_D2.0mm
- TP58: renamed from TP47; footprint (none) -> TestPoint:TestPoint_Pad_D2.0mm
- TP59: renamed from TP49; footprint (none) -> TestPoint:TestPoint_Pad_D2.0mm
- U31: renamed from U27; footprint (none) -> Package_SO:TSSOP-14_4.4x5mm_P0.65mm
- renumbered U29 to U30
Connections:
- net +5V: now also U32.5
- net DRV3_NEG: now also U31.5 (IN2+)
- net DRV4_NEG: now also U31.10 (IN3+)
- net GND: now also U32.2
- net MOS_3: now also U31.6 (IN2-)
- net MOS_4: now also U31.9 (IN3-)
- net DRV1_ADC: now reaches C52.2, R99.2, TP55.1
- net DRV1_ADC: now also U32.1
- net DRV2_ADC: now reaches C54.2, R101.2, TP56.1
- net DRV2_ADC: now also U32.6
- net DRV3_ADC: now reaches C55.2, R103.2, TP57.1
- net DRV3_ADC: now also U32.4
- net DRV4_ADC: now reaches C57.2, R105.2, TP58.1
- net DRV4_ADC: now also U32.3
- net DRV5_ADC: now reaches C58.2, R107.2, TP59.1
- net at R105.1: now also U31.8 (OUT3)
- net at R103.1: now also U31.7 (OUT2)
Other:
- note added: "fc = 1.5kHz"
- note removed: "fc = 2.5kHz"
