File: karca_v2/battery_monitoring.kicad_sch (KiCad schematic)
At the start: 14 parts, among them U24 INA180A2, U25 MCP3202, U26 TLV9301xDBV

Commit message: Version alpha
Parts:
- removed D49, D50: D_Schottky, Diode_SMD:D_SMA, symbol Device:D_Schottky
- removed U25: MCP3202, symbol Analog_ADC:MCP3202
- added C70, C71: 0.1u, Capacitor_SMD:C_0402_1005Metric, symbol Device:C
- added U41: NUP4202, Package_SO:TSOP-6_1.65x3.05mm_P0.95mm, symbol Power_Protection:NUP4202
- added U42: MCP3204, Package_SO:SO-14_3.9x8.65mm_P1.27mm, symbol Analog_ADC:MCP3204
- C60: renamed from C49; footprint Capacitor_SMD:C_1206_3216Metric -> Capacitor_SMD:C_0402_1005Metric
- C61: renamed from C50; value 68n -> 0.1u
- R112: renamed from R96; footprint (none) -> Resistor_SMD:R_1206_3216Metric
- R113: renamed from R97; value 910 -> 1k; footprint (none) -> Resistor_SMD:R_1206_3216Metric
- R114: renamed from R98; footprint (none) -> Resistor_SMD:R_1206_3216Metric
- R115: renamed from R99; footprint (none) -> Resistor_SMD:R_1206_3216Metric
- TP61: renamed from TP43; footprint (none) -> TestPoint:TestPoint_Pad_D2.0mm
- TP62: renamed from TP44; footprint (none) -> TestPoint:TestPoint_Pad_D2.0mm
- renumbered C66 to C59, U24 to U34, U26 to U36
Connections:
- net +5V: now also C70.1, U41.5, U42.13 (Vref), U42.14 (Vdd)
- net BAT_CLK: now also U42.11 (CLK)
- net BAT_MISO: now also U42.10 (Dout)
- net BAT_MOSI: now also U42.9 (Din)
- net CS: now also U42.8 (~{CS}/SHDN)
- net GND: now also C70.2, C71.1, C71.2, U41.2, U42.12 (AGND), U42.7 (DGND)
- net at C61.2, R113.2, TP61.1: now also U41.4, U42.1 (CH0)
- net at TP62.1, U36.1, U36.4 (-): now also U41.3, U42.2 (CH1)
- new net DRV5_ADC: U42.3 (CH2)
- new net DRV5_TVS: U41.6
- no-connect marks 0 -> 2
Other:
- note added: "fc = 1.5kHz"
- note removed: "fc = 2.5kHz"

Commit message: fkkkkkkkkkk
Parts:
- U41: footprint Package_SO:TSOP-6_1.65x3.05mm_P0.95mm -> Package_TO_SOT_SMD:SOT-363_SC-70-6
Changed lines of the file:
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@@
       (effects (font (size 1.27 1.27)) (justify left))
     )
-    (property "Footprint" "Package_SO:TSOP-6_1.65x3.05mm_P0.95mm" (at 161.925 75.565 0)
+    (property "Footprint" "Package_TO_SOT_SMD:SOT-363_SC-70-6" (at 161.925 75.565 0)
       (effects (font (size 1.27 1.27)) hide)
     )
