File: karca_v2/karca_v2.kicad_pcb (KiCad board)
At the start: 4 copper layers, 250 x 145 mm, 361 parts, among them J1 CON_FAN1, J10 Keyhole ignition switch, J11 Screw_Terminal_01x04, J12 Buzzer, J2 Conn_Batt, J3 USB_B_Micro, J4 LoadCell_1_2, J5 LoadCell_3_4, J6 Screw_Terminal_01x08, J7 Raspberry_pi, J8 Screw_Terminal_01x08, J9 Screw_Terminal_01x10, Q1 AO3401A, Q10 IRF3708, Q11 IRF3708, Q12 IRF3708, Q13 IRF3708, Q2 PN2222A, Q4 IRF3708, Q9 IRF3708, SW1 SW_SPST, SW2 SW_SPST, SW3 SW_SPST, U1 TVS1400DRV, U10 NUP4202, U11 M41T93, U12 NUP4202, U13 TLV9304xD, U14 TS5A3159ADBVR, U17 TS5A3159ADBVR, U19 TS5A3159ADBVR, U2 MCP3208, U22 TS5A3159ADBVR, U24 AD8495, U26 AD8495, U27 AD8495, U29 AD8495, U3 NUP4202, U30 INA180A4, U32 NUP4202, U33 AD8223, U34 INA180A2, U35 AD8223, U36 TLV9301xDBV, U4 TLV9304xD, U41 NUP4202, U42 MCP3204, U43 AD8223, U44 AD8223, U5 TLV9304xD, U6 TPS7A24, U7 TLV9304xD, U8 TLV9304xD, U9 MCP3208

Commit message: unrouted adc traces
Parts:
- moved TP39 28.0 mm to (114.1, 116.8)
Routing:
- net /Drivers/IGN_CTL: track 268.0 -> 5.29 mm, vias 1 -> 0
- net /Drivers/IGN_CONT: track 253.9 -> 2.21 mm, vias 1 -> 0
- net /Drivers/DRV2_ADC: track 233.4 -> 22.6 mm, vias 2 -> 1
- net /Drivers/DRV1_CTL: track 205.3 -> 3.45 mm, vias 1 -> 0
- net /Drivers/DRV3_ADC: track 227.3 -> 30.8 mm, vias 2 -> 1
- net /Drivers/DRV4_ADC: track 238.4 -> 44.1 mm
- net /Pressure Transducers/TC_3_ADC: track 257.3 -> 63.0 mm, vias 2 -> 1
- net /Drivers/DRV5_ADC: track 218.9 -> 27.4 mm
- net /Drivers/DRV2_CTL: track 197.1 -> 5.98 mm, vias 1 -> 0
- net /Drivers/DRV4_CTL: track 186.4 -> 5.45 mm, vias 1 -> 0
- net /Pressure Transducers/TC_4_ADC: track 219.6 -> 41.1 mm, vias 2 -> 0
- net /Drivers/DRV5_CTL: track 180.1 -> 5.09 mm, vias 1 -> 0
- net /Drivers/DRV3_CTL: track 179.3 -> 4.62 mm, vias 1 -> 0
- net /Pressure Transducers/TC_1_ADC: track 201.4 -> 31.0 mm, vias 2 -> 0
- net /Pressure Transducers/TC_2_ADC: track 221.0 -> 51.2 mm, vias 2 -> 1
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
Commit message: fkkkkkkkkkk
Parts:
- U10: renamed from U12; footprint Package_SO:TSOP-6_1.65x3.05mm_P0.95mm -> Package_TO_SOT_SMD:SOT-363_SC-70-6
- U3, U32, U41: footprint Package_SO:TSOP-6_1.65x3.05mm_P0.95mm -> Package_TO_SOT_SMD:SOT-363_SC-70-6
- moved C5 147.0 mm to (190.4, 146.2)
- moved U9 147.0 mm to (187.2, 141.1)
- moved TP57 146.5 mm to (199.2, 132.7)
- moved TP56 141.9 mm to (195.2, 132.6)
- moved U12 141.2 mm to (184.3, 126.1)
- moved TP12 141.2 mm to (185.3, 134.1)
- moved TP19 140.6 mm to (171.8, 133.8)
- moved TP13 140.6 mm to (181.1, 132.6)
- moved TP21 139.2 mm to (168.8, 131.3)
- moved TP58 138.0 mm to (188.8, 130.2)
- moved TP55 134.8 mm to (191.3, 132.5)
- moved TP10 134.2 mm to (179.7, 129.7)
- moved U32 133.0 mm to (191.6, 126.9)
- moved TP11 131.4 mm to (179.3, 138.0)
- moved TP17 130.5 mm to (161.8, 129.7)
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- renumbered U10 to U12
Connections:
- C52 pad 2: /Drivers/DRV1_ADC -> /DRV1_ADC
- C54 pad 2: /Drivers/DRV2_ADC -> /DRV2_ADC
- C55 pad 2: /Drivers/DRV3_ADC -> /DRV3_ADC
- C57 pad 2: /Drivers/DRV4_ADC -> /DRV4_ADC
- Ce1 pad 1: /Pressure Transducers/TC_1_ADC -> /Load Cells/TC_1_ADC
- Ce2 pad 1: /Pressure Transducers/TC_2_ADC -> /Load Cells/TC_2_ADC
- Ce3 pad 1: /Pressure Transducers/TC_3_ADC -> /Load Cells/TC_3_ADC
- Ce4 pad 1: /Pressure Transducers/TC_4_ADC -> /Load Cells/TC_4_ADC
- D4 pad 2: +5V -> Net-(D4-A)
- J3 pad 1: +5V -> Net-(D4-A)
- J7 pad 29: Net-(J7-Pin_29) -> unconnected-(J7-Pin_29-Pad29)
- J7 pad 3: unconnected-(J7-Pin_3-Pad3) -> Net-(J7-Pin_3)
- Q1 pad 1: +5V -> Net-(D4-A)
- R10 pad 2: Net-(J7-Pin_29) -> Net-(J7-Pin_3)
- R101 pad 2: /Drivers/DRV2_ADC -> /DRV2_ADC
- R103 pad 2: /Drivers/DRV3_ADC -> /DRV3_ADC
- R105 pad 2: /Drivers/DRV4_ADC -> /DRV4_ADC
- R11 pad 2: Net-(J7-Pin_29) -> Net-(J7-Pin_3)
- R99 pad 2: /Drivers/DRV1_ADC -> /DRV1_ADC
- TP14 pad 1: /Pressure Transducers/TC_1_ADC -> /Load Cells/TC_1_ADC
- TP15 pad 1: /Pressure Transducers/TC_1_ADC -> /Load Cells/TC_1_ADC
- TP16 pad 1: /Pressure Transducers/TC_2_ADC -> /Load Cells/TC_2_ADC
- TP17 pad 1: /Pressure Transducers/TC_2_ADC -> /Load Cells/TC_2_ADC
- TP18 pad 1: /Pressure Transducers/TC_3_ADC -> /Load Cells/TC_3_ADC
- TP19 pad 1: /Pressure Transducers/TC_3_ADC -> /Load Cells/TC_3_ADC
- TP20 pad 1: /Pressure Transducers/TC_4_ADC -> /Load Cells/TC_4_ADC
- TP21 pad 1: /Pressure Transducers/TC_4_ADC -> /Load Cells/TC_4_ADC
- TP5 pad 1: +5V -> Net-(D4-A)
- TP55 pad 1: /Drivers/DRV1_ADC -> /DRV1_ADC
- TP56 pad 1: /Drivers/DRV2_ADC -> /DRV2_ADC
- TP57 pad 1: /Drivers/DRV3_ADC -> /DRV3_ADC
- TP58 pad 1: /Drivers/DRV4_ADC -> /DRV4_ADC
- U10 pad 1: /Pressure Transducers/TC_4_ADC -> /Load Cells/TC_1_ADC
- U10 pad 3: /Pressure Transducers/TC_3_ADC -> /Load Cells/TC_2_ADC
- U10 pad 4: /Pressure Transducers/TC_2_ADC -> /Load Cells/TC_3_ADC
- U10 pad 6: /Pressure Transducers/TC_1_ADC -> /Load Cells/TC_4_ADC
- U12 pad 1: /Pressure Transducers/pt_circuitry3/OUT -> /Pressure Transducers/pt_circuitry/OUT
- U12 pad 3: /Pressure Transducers/pt_circuitry2/OUT -> /Pressure Transducers/pt_circuitry1/OUT
- U12 pad 4: /Pressure Transducers/pt_circuitry1/OUT -> /Pressure Transducers/pt_circuitry2/OUT
- U12 pad 6: /Pressure Transducers/pt_circuitry/OUT -> /Pressure Transducers/pt_circuitry3/OUT
- U13 pad 1: /Pressure Transducers/TC_2_ADC -> /Load Cells/TC_2_ADC
- U13 pad 13: /Pressure Transducers/TC_3_ADC -> /Load Cells/TC_3_ADC
- U13 pad 14: /Pressure Transducers/TC_3_ADC -> /Load Cells/TC_3_ADC
- U13 pad 2: /Pressure Transducers/TC_2_ADC -> /Load Cells/TC_2_ADC
- U13 pad 6: /Pressure Transducers/TC_1_ADC -> /Load Cells/TC_1_ADC
- U13 pad 7: /Pressure Transducers/TC_1_ADC -> /Load Cells/TC_1_ADC
- U13 pad 8: /Pressure Transducers/TC_4_ADC -> /Load Cells/TC_4_ADC
- U13 pad 9: /Pressure Transducers/TC_4_ADC -> /Load Cells/TC_4_ADC
- U2 pad 1: /Load Cells/LC_Amplification/OUT -> /Load Cells/TC_3_ADC
- U2 pad 2: /Load Cells/LC_Amplification1/OUT -> /Load Cells/TC_4_ADC
- U2 pad 3: /Load Cells/LC_Amplification2/OUT -> /Load Cells/TC_1_ADC
- U2 pad 4: /Load Cells/LC_Amplification3/OUT -> /Load Cells/TC_2_ADC
- U2 pad 5: /Drivers/DRV1_ADC -> /Load Cells/LC_Amplification/OUT
- U2 pad 6: /Drivers/DRV2_ADC -> /Load Cells/LC_Amplification1/OUT
- U2 pad 7: /Drivers/DRV3_ADC -> /Load Cells/LC_Amplification2/OUT
- U2 pad 8: /Drivers/DRV4_ADC -> /Load Cells/LC_Amplification3/OUT
- U3 pad 4: /Load Cells/LC_Amplification1/OUT -> /Load Cells/LC_Amplification/OUT
- U3 pad 6: /Load Cells/LC_Amplification/OUT -> /Load Cells/LC_Amplification1/OUT
- U32 pad 1: /Drivers/DRV1_ADC -> /DRV3_ADC
- U32 pad 3: /Drivers/DRV4_ADC -> /DRV2_ADC
- U32 pad 4: /Drivers/DRV3_ADC -> /DRV1_ADC
- U32 pad 6: /Drivers/DRV2_ADC -> /DRV4_ADC
- U9 pad 1: /Pressure Transducers/pt_circuitry/OUT -> /DRV3_ADC
- U9 pad 2: /Pressure Transducers/pt_circuitry1/OUT -> /DRV2_ADC
- U9 pad 3: /Pressure Transducers/pt_circuitry2/OUT -> /DRV1_ADC
- U9 pad 4: /Pressure Transducers/pt_circuitry3/OUT -> /DRV4_ADC
- U9 pad 5: /Pressure Transducers/TC_1_ADC -> /Pressure Transducers/pt_circuitry2/OUT
- U9 pad 6: /Pressure Transducers/TC_2_ADC -> /Pressure Transducers/pt_circuitry3/OUT
- U9 pad 7: /Pressure Transducers/TC_3_ADC -> /Pressure Transducers/pt_circuitry/OUT
- U9 pad 8: /Pressure Transducers/TC_4_ADC -> /Pressure Transducers/pt_circuitry1/OUT
Routing:
- net /Drivers/IGN_CTL: track 5.29 -> 239.0 mm
- net /Load Cells/LC_SELECTOR: track 0.00 -> 194.8 mm, vias 0 -> 4
- net /Drivers/DRV5_ADC: track 27.4 -> 167.9 mm
- net /Drivers/IGN_CONT: track 2.21 -> 134.1 mm, vias 0 -> 2
- net /Load Cells/TC_2_ADC: track 0.00 -> 97.3 mm
- net /Drivers/DRV1_CTL: track 3.45 -> 100.4 mm
- net /DRV2_ADC: track 0.00 -> 93.5 mm, vias 0 -> 2
- net Net-(U42-CH0): track 21.7 -> 115.0 mm, vias 1 -> 2
- net /Load Cells/TC_3_ADC: track 0.00 -> 91.8 mm
- net /DRV4_ADC: track 0.00 -> 90.9 mm, vias 0 -> 2
- net /SPI.MOSI: track 54.2 -> 143.4 mm
- net /SPI.CLK: track 45.4 -> 132.0 mm
- net /Drivers/DRV2_CTL: track 5.98 -> 88.6 mm
- net /DRV3_ADC: track 0.00 -> 79.7 mm, vias 0 -> 2
- net /Drivers/DRV3_CTL: track 4.62 -> 74.0 mm
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- added copper zone on F.Cu, net +12V
