File: karca_v2/regulators.kicad_sch (KiCad schematic)
At the start: 29 parts, among them J1 CON_FAN1, J2 Screw_Terminal_01x02, SW1 SW_SPST, SW2 SW_SPST, U1 TPS565208, U2 TPS7A57

Commit message: modified sch
Parts:
- added D25: LED, LED_SMD:LED_1206_3216Metric, symbol Device:LED
- added R93: 600, symbol Device:R_US
- R1: value R -> 600
Connections:
- net +12V: now also TP2.1; no longer D1.1 (K)
- net GND: now also D25.2 (A)
- net battery_monitoring/Battery+: now also R93.2
- net at J2.2 (Pin_2): now also D1.2 (A); no longer F1.1
- removed net battery_monitoring/Load+: D1.2 (A), TP2.1
- new net: D25.1 (K), R93.1
- new net: D1.1 (K), F1.1
Other:
- note added: "reverse polarity indicator LED"
- moved on the sheet: TP3

Commit message: updated
Parts:
- removed D1: 1N5822RLG, Diode_THT:D_DO-201AD_P15.24mm_Horizontal, symbol Device:D
- removed D25: LED, LED_SMD:LED_1206_3216Metric, symbol Device:LED
- removed R93: 600, symbol Device:R_US
- added C46: 10u, symbol Device:C
- added D24: D_Schottky, symbol Device:D_Schottky
- added D48: 1N5822RLG, Diode_THT:D_DO-201AD_P15.24mm_Horizontal, symbol Device:D
- added D66: LED, LED_SMD:LED_1206_3216Metric, symbol Device:LED
- added J11: USB_B_Micro, symbol Connector:USB_B_Micro
- added MD1: OKL-T_6-W12N-C, OKL-T_6-W12N-C:MURATA_OKL-T-6-W12N-C_0, symbol OKL-T/6-W12N-C:OKL-T_6-W12N-C
- added Q8: AO3401A, symbol Simulation_SPICE:PMOS
- added R114: 1.5k, symbol Device:R_US
- added R117: 1.34k, symbol Device:R_US
- added R65: 10k, symbol Device:R_US
- added SW3: SW_SPST, symbol Switch:SW_SPST
- added U55: TVS1400DRV, Package_SON:WSON-6-1EP_2x2mm_P0.65mm_EP1x1.6mm, symbol Power_Protection:TVS1400DRV
- R1: value 600 -> 470
Connections:
- net +12V: now also D66.2 (A), SW3.1 (A)
- net +5V: now also D24.1 (K), D24.2 (A), J11.1 (VBUS), MD1.4 (VOUT), Q8.1 (D), Q8.2 (G), Q8.3 (S), R65.1
- net GND: now also C46.2, J11.5 (GND), J11.6 (Shield), MD1.3 (1_GROUND), MD1.7 (2_GROUND), R117.2, R65.2, U55.1 (GND), U55.2 (GND), U55.3 (GND), U55.7 (GND)
- net battery_monitoring/Battery+: now also D48.1 (K), U55.4 (IN), U55.5 (IN), U55.6 (IN); no longer SW2.2 (B)
- net at J2.2 (Pin_2): now also F1.1
- new net: C46.1, MD1.2 (VIN), SW3.2 (B)
- new net: MD1.6 (TRIM), R117.1
- new net: D48.2 (A), SW2.2 (B)
- new net: D66.1 (K), R114.1
- new net: MD1.10 (POWER_GOOD_OUT), R114.2
- no-connect marks 1 -> 10
Other:
- note added: "14V Vrwm surge protection diode"
- note added: "Active Low pin"
- note added: "Power path management (allows USB power)"
- note added: "Red LED indicates 5V regulator is off/malfunctioning"
- note added: "When battery/12V power supply is connected, P-MOS gate is pulled high, turning it off. This disconnects USB power"
- note removed: "reverse polarity indicator LED"
- moved on the sheet: F1, J2, SW2, TP3

Commit message: Version alpha
Parts:
- removed C1, C52, C53: 10u, symbol Device:C
- removed C2, C51: 0.1u, symbol Device:C
- removed C54, C55, C57: 22u, symbol Device:C
- removed C56: 4.7u, symbol Device:C
- removed D66: LED, LED_SMD:LED_1206_3216Metric, symbol Device:LED
- removed L1: 3.3u, symbol Device:L
- removed R101: 100k, symbol Device:R_US
- removed R102: 50k, symbol Device:R_US
- removed R114: 1.5k, symbol Device:R_US
- removed R2: 10k, symbol Device:R_US
- removed R4: 62k, symbol Device:R_US
- removed U1: TPS565208, Package_TO_SOT_SMD:SOT-23-6, symbol Regulator_Switching:TPS565208
- removed U2: TPS7A57, symbol karca_lib:TPS7A57
- added C72: 10u, Capacitor_SMD:C_1206_3216Metric, symbol Device:C
- added D4: LED, LED_SMD:LED_1206_3216Metric, symbol Device:LED
- added R3: 250, Resistor_SMD:R_1206_3216Metric, symbol Device:R_US
- added TP4, TP5: TestPoint, TestPoint:TestPoint_Pad_D2.0mm, symbol Connector:TestPoint
- C1: renamed from C46; footprint (none) -> Capacitor_Tantalum_SMD:CP_EIA-3216-18_Kemet-A
- D3: value RED -> LED; footprint (none) -> LED_SMD:LED_1206_3216Metric
- D5: renamed from D24; footprint (none) -> Diode_SMD:D_SMA
- F1: footprint (none) -> 4628:FUSE_4628
- J1: footprint (none) -> terminal blocks:P-2604-1102
- J2: value Screw_Terminal_01x02 -> Conn_Batt; footprint (none) -> terminal blocks:P-2604-1102
- J3: renamed from J11; footprint (none) -> USB-B:GCT_USB3130-XX-X_REVD
- MD1: footprint OKL-T_6-W12N-C:MURATA_OKL-T-6-W12N-C_0 -> OKL-T6-W12N:MURATA_OKL-T-6-W12N-C_0
- Q1: renamed from Q8; footprint (none) -> AO3401A:SOT23-3
- R1: footprint (none) -> Resistor_SMD:R_1206_3216Metric
- R2: renamed from R65; footprint (none) -> Resistor_SMD:R_1206_3216Metric
- R4: renamed from R117; footprint (none) -> Resistor_SMD:R_1206_3216Metric
- R5: value 330 -> 250; footprint (none) -> Resistor_SMD:R_1206_3216Metric
- SW1, SW2, SW3: footprint (none) -> 500SSP1S2M2QEA:SW_500SSP1S2M2QEA
- TP1, TP2, TP3: footprint (none) -> TestPoint:TestPoint_Pad_D2.0mm
- renumbered D48 to D1, U55 to U1
Connections:
- net +5V: now also C72.1, D4.2 (A), TP4.1, TP5.1
- net GND: now also R5.2, C72.2, R3.2; no longer R5.1
- net at D3.1 (K): now also R3.1; no longer R5.2
- new net: D4.1 (K), R5.1
Other:
- sheet battery_monitoring ports: added DRV5_ADC, DRV5_TVS; removed none
- note removed: "Buck converter: Minimizes power dissipation (12V to 5.5V) LDO: reduces output ripple from Buck (5.5V to 5V)"
- note removed: "Iout(max) =5A"
- note removed: "PG pin can be left floating if we don't need this feature"
- note removed: "Red LED indicates 5V regulator is off/malfunctioning"
- note removed: "Vout = 5.5V = 0.76*(1+(R4/R2))"
- note removed: "Vout = 5V = Rref*Iref = 100k*50u"
- moved on the sheet: C1, D1, D2, D5, F1, J1, J2, J3, MD1, Q1, R1, R2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

Commit message: fkkkkkkkkkk
Connections:
- net +5V: no longer D4.2 (A), J3.1 (VBUS), Q1.1 (D), TP5.1
- new net: D4.2 (A), J3.1 (VBUS), Q1.1 (D), TP5.1
Changed lines of the file:
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@@
   (junction (at 347.726 165.481) (diameter 0) (color 0 0 0 0)
-  )
-  (junction (at 357.505 146.05) (diameter 0) (color 0 0 0 0)
   )
   (junction (at 287.909 135.89) (diameter 0) (color 0 0 0 0)
@@
         )
       )
-    )
-  )
-  (symbol (lib_id "power:+5V") (at 357.505 146.05 0) (unit 1)
-    (in_bom yes) (on_board yes) (dnp no) (fields_autoplaced)
-    (property "Reference" "#PWR0203" (at 357.505 149.86 0)
-      (effects (font (size 1.27 1.27)) hide)
-    )
-    (property "Value" "+5V" (at 357.505 140.97 0)
-      (effects (font (size 1.27 1.27)))
-    )
-    (property "Footprint" "" (at 357.505 146.05 0)
-      (effects (font (size 1.27 1.27)) hide)
-    )
-    (property "Datasheet" "" (at 357.505 146.05 0)
-      (effects (font (size 1.27 1.27)) hide)
-    )
-    (pin "1")
-    (instances
-      (project "karca_v2"
-        (path "/29cf4797-56f2-4f57-ae95-7df639362e3c/d3760e06-a79f-4c5f-b008-48bf6f5622ff"
-          (reference "#PWR0203") (unit 1)
-        )
-      )

Commit message: discrete traces
Parts:
- renumbered C72 to C2
Changed lines of the file:
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@@
   (symbol (lib_id "power:GND") (at 347.726 165.481 0) (unit 1)
     (in_bom yes) (on_board yes) (dnp no) (fields_autoplaced)
-    (property "Reference" "#PWR012" (at 347.726 171.831 0)
+    (property "Reference" "#PWR013" (at 347.726 171.831 0)
       (effects (font (size 1.27 1.27)) hide)
     )
@@
       (project "karca_v2"
         (path "/29cf4797-56f2-4f57-ae95-7df639362e3c/d3760e06-a79f-4c5f-b008-48bf6f5622ff"
-          (reference "#PWR012") (unit 1)
+          (reference "#PWR013") (unit 1)
         )
       )
@@
   (symbol (lib_id "power:GND") (at 368.681 170.434 0) (unit 1)
     (in_bom yes) (on_board yes) (dnp no)
-    (property "Reference" "#PWR013" (at 368.681 176.784 0)
+    (property "Reference" "#PWR014" (at 368.681 176.784 0)
       (effects (font (size 1.27 1.27)) hide)
     )
@@
       (project "karca_v2"
         (path "/29cf4797-56f2-4f57-ae95-7df639362e3c/d3760e06-a79f-4c5f-b008-48bf6f5622ff"
-          (reference "#PWR013") (unit 1)
+          (reference "#PWR014") (unit 1)
         )
       )
@@
   (symbol (lib_id "power:GND") (at 361.061 156.464 0) (unit 1)
     (in_bom yes) (on_board yes) (dnp no) (fields_autoplaced)
-    (property "Reference" "#PWR09" (at 361.061 162.814 0)
+    (property "Reference" "#PWR010" (at 361.061 162.814 0)
       (effects (font (size 1.27 1.27)) hide)
     )
@@
       (project "karca_v2"
         (path "/29cf4797-56f2-4f57-ae95-7df639362e3c/d3760e06-a79f-4c5f-b008-48bf6f5622ff"
-          (reference "#PWR09") (unit 1)
+          (reference "#PWR010") (unit 1)
         )
       )
@@
   (symbol (lib_id "Device:C") (at 286.385 141.605 0) (unit 1)
     (in_bom yes) (on_board yes) (dnp no)
-    (property "Reference" "C72" (at 287.655 139.065 0)
+    (property "Reference" "C2" (at 287.655 139.065 0)
       (effects (font (size 1.27 1.27)) (justify left))
     )
@@
       (project "karca_v2"
         (path "/29cf4797-56f2-4f57-ae95-7df639362e3c/d3760e06-a79f-4c5f-b008-48bf6f5622ff"
-          (reference "C72") (unit 1)
+          (reference "C2") (unit 1)
         )
       )
@@
   (symbol (lib_id "power:GND") (at 286.385 145.415 0) (unit 1)
     (in_bom yes) (on_board yes) (dnp no) (fields_autoplaced)
-    (property "Reference" "#PWR0199" (at 286.385 151.765 0)
+    (property "Reference" "#PWR08" (at 286.385 151.765 0)
       (effects (font (size 1.27 1.27)) hide)
     )
@@
       (project "karca_v2"
         (path "/29cf4797-56f2-4f57-ae95-7df639362e3c/d3760e06-a79f-4c5f-b008-48bf6f5622ff"
-          (reference "#PWR0199") (unit 1)
+          (reference "#PWR08") (unit 1)
         )
       )
@@
   (symbol (lib_id "power:GND") (at 286.131 161.29 0) (unit 1)
     (in_bom yes) (on_board yes) (dnp no) (fields_autoplaced)
-    (property "Reference" "#PWR011" (at 286.131 167.64 0)
+    (property "Reference" "#PWR012" (at 286.131 167.64 0)
       (effects (font (size 1.27 1.27)) hide)
     )
@@
       (project "karca_v2"
         (path "/29cf4797-56f2-4f57-ae95-7df639362e3c/d3760e06-a79f-4c5f-b008-48bf6f5622ff"
-          (reference "#PWR011") (unit 1)
+          (reference "#PWR012") (unit 1)
         )
       )
@@
   (symbol (lib_id "power:GND") (at 319.278 160.02 0) (unit 1)
     (in_bom yes) (on_board yes) (dnp no)
-    (property "Reference" "#PWR010" (at 319.278 166.37 0)
+    (property "Reference" "#PWR011" (at 319.278 166.37 0)
       (effects (font (size 1.27 1.27)) hide)
     )
@@
       (project "karca_v2"
         (path "/29cf4797-56f2-4f57-ae95-7df639362e3c/d3760e06-a79f-4c5f-b008-48bf6f5622ff"
-          (reference "#PWR010") (unit 1)
+          (reference "#PWR011") (unit 1)
         )
       )
@@
   (symbol (lib_id "power:+5V") (at 402.209 152.273 0) (unit 1)
     (in_bom yes) (on_board yes) (dnp no) (fields_autoplaced)
-    (property "Reference" "#PWR08" (at 402.209 156.083 0)
+    (property "Reference" "#PWR09" (at 402.209 156.083 0)
       (effects (font (size 1.27 1.27)) hide)
     )
@@
       (project "karca_v2"
         (path "/29cf4797-56f2-4f57-ae95-7df639362e3c/d3760e06-a79f-4c5f-b008-48bf6f5622ff"
-          (reference "#PWR08") (unit 1)
-        )
-      )
+          (reference "#PWR09") (unit 1)
+        )
+      )

Commit message: fixed violations
Parts:
- J3: footprint USB-B:GCT_USB3130-XX-X_REVD -> USB-B:GCT_USB3090-XX-X_REVE
Connections:
- net +5V: no longer C2.1, D3.2 (A), D5.2 (A), MD1.4 (VOUT), Q1.2 (G), R2.1, TP4.1
- new net BAT_OUT: C2.1, D3.2 (A), D5.2 (A), MD1.4 (VOUT), Q1.2 (G), R2.1, TP4.1
Other:
- moved on the sheet: D4, D5, J3, Q1, R2, R5, TP5

Commit message: save before rerouting
Connections:
- net BAT_OUT: now also Q1.1 (G); no longer Q1.2 (G)
- net at D4.2 (A), J3.1 (VBUS), TP5.1: now also Q1.2 (S); no longer Q1.1 (D)
Other:
- moved on the sheet: Q1
Changed lines of the file:
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@@
     )
   )
-  (symbol (lib_id "Simulation_SPICE:PMOS") (at 381 157.48 90) (mirror x) (unit 1)
+  (symbol (lib_id "Simulation_SPICE:PMOS") (at 381 157.48 270) (unit 1)
     (in_bom yes) (on_board yes) (dnp no)
     (property "Reference" "Q1" (at 381 163.957 90)
@@
       (effects (font (size 1.27 1.27)))
     )
-    (property "Footprint" "AO3401A:SOT23-3" (at 378.46 162.56 0)
+    (property "Footprint" "AO3401A:SOT23-3" (at 383.54 162.56 0)
       (effects (font (size 1.27 1.27)) hide)
     )
-    (property "Datasheet" "https://ngspice.sourceforge.io/docs/ngspice-manual.pdf" (at 393.7 157.48 0)
+    (property "Datasheet" "https://ngspice.sourceforge.io/docs/ngspice-manual.pdf" (at 368.3 157.48 0)
       (effects (font (size 1.27 1.27)) hide)
     )
-    (property "Sim.Device" "PMOS" (at 398.145 157.48 0)
+    (property "Sim.Device" "PMOS" (at 363.855 157.48 0)
       (effects (font (size 1.27 1.27)) hide)
     )
-    (property "Sim.Type" "VDMOS" (at 400.05 157.48 0)
+    (property "Sim.Type" "VDMOS" (at 361.95 157.48 0)
       (effects (font (size 1.27 1.27)) hide)
     )
-    (property "Sim.Pins" "1=D 2=G 3=S" (at 396.24 157.48 0)
+    (property "Sim.Pins" "1=D 2=G 3=S" (at 365.76 157.48 0)
       (effects (font (size 1.27 1.27)) hide)
     )
