File: karca_v2/raspberry_pi.kicad_sch (KiCad schematic)
At the start: 10 parts, among them J6 Raspberry_pi, Q1 PN2222A, U7 MT41T93, Y1 32k

Commit message: Version alpha
Parts:
- removed C16: 1u, Capacitor_SMD:C_1206_3216Metric, symbol Device:C
- removed R26, R27: 10k, symbol Device:R_US
- removed U7: MT41T93, symbol karca_lib:M41T93
- removed Y1: 32k, symbol Device:Crystal
- added C6: 1u, Capacitor_SMD:C_1206_3216Metric, symbol Device:C
- added R8, R9: 10k, Resistor_SMD:R_1206_3216Metric, symbol Device:R_US
- added U11: M41T93, Package_SO:SOIC-18W_7.5x11.6mm_P1.27mm, symbol karca_lib:M41T93
- J7: renamed from J6; footprint (none) -> Connector_PinHeader_2.00mm:PinHeader_2x20_P2.00mm_Vertical
- R10: renamed from R28; footprint (none) -> Resistor_SMD:R_1206_3216Metric
- R11: renamed from R29; footprint (none) -> Resistor_SMD:R_1206_3216Metric
- renumbered D12 to D6, Q1 to Q2
Connections:
- net +5V: now also R8.1, R9.1, U11.15 (VCC), U11.6 (DU)
- net GND: now also C6.1, U11.16 (NF), U11.2 (NF), U11.9 (VSS)
- net RTC_CS: now also J7.37 (Pin_37), U11.14 (E); no longer J7.32 (Pin_32)
- net RTC_IRQ: now also J7.38 (Pin_38), R8.2, U11.12 (IRQ); no longer J7.36 (Pin_36)
- net SPI.CLK: now also U11.11 (SCL)
- net SPI.MISO: now also U11.13 (SDO)
- net SPI.MOSI: now also U11.10 (SDI)
- net ADC_DRV_CS: no longer names the net of J7.28 (Pin_28)
- new net: R9.2, U11.5 (RST)
- new net: C6.2, U11.8 (VBAT)
- no-connect marks 14 -> 16
Other:
- note removed: "12.5pF load capacitance"

Commit message: fkkkkkkkkkk
Connections:
- net at R10.2, R11.2: now also J7.3 (Pin_3); no longer J7.29 (Pin_29)
Other:
- moved on the sheet: D6, Q2, R10, R11
Changed lines of the file:
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@@
   (junction (at 160.02 60.96) (diameter 0) (color 0 0 0 0)
   )
+  (junction (at 108.585 60.96) (diameter 0) (color 0 0 0 0)
+  )
   (junction (at 121.92 91.44) (diameter 0) (color 0 0 0 0)
   )
@@
   (junction (at 121.92 109.22) (diameter 0) (color 0 0 0 0)
   )
-  (junction (at 113.03 96.52) (diameter 0) (color 0 0 0 0)
-  )
   (junction (at 215.9 60.96) (diameter 0) (color 0 0 0 0)
   )
@@
   (junction (at 195.58 60.96) (diameter 0) (color 0 0 0 0)
   )
-  (junction (at 92.71 114.3) (diameter 0) (color 0 0 0 0)
+  (junction (at 88.265 78.74) (diameter 0) (color 0 0 0 0)
   )
   (no_connect (at 151.13 73.66))
+  (no_connect (at 138.43 96.52))
   (no_connect (at 198.12 71.12))
   (no_connect (at 151.13 104.14))
-  (no_connect (at 138.43 63.5))
   (no_connect (at 138.43 68.58))
   (no_connect (at 151.13 83.82))
@@
     (stroke (width 0) (type default))
   )
+  (wire (pts (xy 109.855 63.5) (xy 109.855 60.96))
+    (stroke (width 0) (type default))
+  )
   (wire (pts (xy 160.02 63.5) (xy 160.02 60.96))
     (stroke (width 0) (type default))
   )
-  (wire (pts (xy 113.03 96.52) (xy 113.03 100.33))
+  (wire (pts (xy 108.585 60.96) (xy 108.585 64.77))
     (stroke (width 0) (type default))
   )
@@
     (stroke (width 0) (type default))
   )
-  (wire (pts (xy 100.33 96.52) (xy 102.87 96.52))
+  (wire (pts (xy 95.885 60.96) (xy 98.425 60.96))
     (stroke (width 0) (type default))
   )
@@
     (stroke (width 0) (type default))
   )
-  (wire (pts (xy 92.71 111.76) (xy 92.71 114.3))
-    (stroke (width 0) (type default))
-  )
-  (wire (pts (xy 92.71 114.3) (xy 92.71 116.84))
+  (wire (pts (xy 88.265 76.2) (xy 88.265 78.74))
+    (stroke (width 0) (type default))
+  )
+  (wire (pts (xy 88.265 78.74) (xy 88.265 81.28))
     (stroke (width 0) (type default))
   )
@@
     (stroke (width 0) (type default))
   )
-  (wire (pts (xy 113.03 114.3) (xy 92.71 114.3))
-    (stroke (width 0) (type default))
-  )
-  (wire (pts (xy 113.03 107.95) (xy 113.03 114.3))
+  (wire (pts (xy 108.585 78.74) (xy 88.265 78.74))
+    (stroke (width 0) (type default))
+  )
+  (wire (pts (xy 108.585 72.39) (xy 108.585 78.74))
     (stroke (width 0) (type default))
   )
@@
     (stroke (width 0) (type default))
   )
+  (wire (pts (xy 109.855 60.96) (xy 108.585 60.96))
+    (stroke (width 0) (type default))
+  )
   (wire (pts (xy 121.92 91.44) (xy 138.43 91.44))
     (stroke (width 0) (type default))
@@
     (stroke (width 0) (type default))
   )
-  (wire (pts (xy 113.03 96.52) (xy 110.49 96.52))
+  (wire (pts (xy 108.585 60.96) (xy 106.045 60.96))
     (stroke (width 0) (type default))
   )
@@
     (stroke (width 0) (type default))
   )
-  (wire (pts (xy 92.71 101.6) (xy 92.71 104.14))
+  (wire (pts (xy 88.265 66.04) (xy 88.265 68.58))
     (stroke (width 0) (type default))
   )
@@
     (stroke (width 0) (type default))
   )
-  (wire (pts (xy 92.71 83.82) (xy 92.71 91.44))
+  (wire (pts (xy 88.265 48.26) (xy 88.265 55.88))
     (stroke (width 0) (type default))
   )
@@
     (stroke (width 0) (type default))
   )
-  (wire (pts (xy 113.03 96.52) (xy 138.43 96.52))
-    (stroke (width 0) (type default))
-  )
   (wire (pts (xy 198.12 76.2) (xy 195.58 76.2))
     (stroke (width 0) (type default))
@@
   )
   (wire (pts (xy 121.92 109.22) (xy 121.92 115.57))
+    (stroke (width 0) (type default))
+  )
+  (wire (pts (xy 138.43 63.5) (xy 109.855 63.5))
     (stroke (width 0) (type default))
   )
@@
     )
   )
-  (symbol (lib_id "Device:R_US") (at 113.03 104.14 180) (unit 1)
-    (in_bom yes) (on_board yes) (dnp no) (fields_autoplaced)
-    (property "Reference" "R11" (at 115.57 102.87 0)
+  (symbol (lib_id "Device:R_US") (at 108.585 68.58 180) (unit 1)
+    (in_bom yes) (on_board yes) (dnp no) (fields_autoplaced)
+    (property "Reference" "R11" (at 111.125 67.31 0)
       (effects (font (size 1.27 1.27)) (justify right))
     )
-    (property "Value" "10k" (at 115.57 105.41 0)
+    (property "Value" "10k" (at 111.125 69.85 0)
       (effects (font (size 1.27 1.27)) (justify right))
     )
-    (property "Footprint" "Resistor_SMD:R_1206_3216Metric" (at 112.014 103.886 90)
-      (effects (font (size 1.27 1.27)) hide)
-    )
-    (property "Datasheet" "~" (at 113.03 104.14 0)
+    (property "Footprint" "Resistor_SMD:R_1206_3216Metric" (at 107.569 68.326 90)
+      (effects (font (size 1.27 1.27)) hide)
+    )
+    (property "Datasheet" "~" (at 108.585 68.58 0)
       (effects (font (size 1.27 1.27)) hide)
     )
@@
     )
   )
-  (symbol (lib_id "Device:R_US") (at 106.68 96.52 90) (unit 1)
+  (symbol (lib_id "Device:R_US") (at 102.235 60.96 90) (unit 1)
     (in_bom yes) (on_board yes) (dnp no)
-    (property "Reference" "R10" (at 106.68 92.71 90)
-      (effects (font (size 1.27 1.27)))
-    )
-    (property "Value" "1k" (at 106.68 93.98 90)
-      (effects (font (size 1.27 1.27)))
-    )
-    (property "Footprint" "Resistor_SMD:R_1206_3216Metric" (at 106.934 95.504 90)
-      (effects (font (size 1.27 1.27)) hide)
-    )
-    (property "Datasheet" "~" (at 106.68 96.52 0)
+    (property "Reference" "R10" (at 102.235 57.15 90)
+      (effects (font (size 1.27 1.27)))
+    )
+    (property "Value" "1k" (at 102.235 58.42 90)
+      (effects (font (size 1.27 1.27)))
+    )
+    (property "Footprint" "Resistor_SMD:R_1206_3216Metric" (at 102.489 59.944 90)
+      (effects (font (size 1.27 1.27)) hide)
+    )
+    (property "Datasheet" "~" (at 102.235 60.96 0)
       (effects (font (size 1.27 1.27)) hide)
     )
@@
     )
   )
-  (symbol (lib_id "Device:LED") (at 92.71 107.95 90) (unit 1)
-    (in_bom yes) (on_board yes) (dnp no) (fields_autoplaced)
-    (property "Reference" "D6" (at 96.52 108.2675 90)
+  (symbol (lib_id "Device:LED") (at 88.265 72.39 90) (unit 1)
+    (in_bom yes) (on_board yes) (dnp no) (fields_autoplaced)
+    (property "Reference" "D6" (at 92.075 72.7075 90)
       (effects (font (size 1.27 1.27)) (justify right))
     )
-    (property "Value" "HBT" (at 96.52 110.8075 90)
+    (property "Value" "HBT" (at 92.075 75.2475 90)
       (effects (font (size 1.27 1.27)) (justify right))
     )
-    (property "Footprint" "LED_SMD:LED_1206_3216Metric" (at 92.71 107.95 0)
-      (effects (font (size 1.27 1.27)) hide)
-    )
-    (property "Datasheet" "~" (at 92.71 107.95 0)
+    (property "Footprint" "LED_SMD:LED_1206_3216Metric" (at 88.265 72.39 0)
+      (effects (font (size 1.27 1.27)) hide)
+    )
+    (property "Datasheet" "~" (at 88.265 72.39 0)
       (effects (font (size 1.27 1.27)) hide)
     )
@@
     )
   )
-  (symbol (lib_id "Transistor_BJT:PN2222A") (at 95.25 96.52 0) (mirror y) (unit 1)
+  (symbol (lib_id "Transistor_BJT:PN2222A") (at 90.805 60.96 0) (mirror y) (unit 1)
     (in_bom yes) (on_board yes) (dnp no)
-    (property "Reference" "Q2" (at 90.17 97.79 0)
+    (property "Reference" "Q2" (at 85.725 62.23 0)
       (effects (font (size 1.27 1.27)) (justify left))
     )
-    (property "Value" "PN2222A" (at 90.17 95.25 0)
+    (property "Value" "PN2222A" (at 85.725 59.69 0)
       (effects (font (size 1.27 1.27)) (justify left))
     )
-    (property "Footprint" "Package_TO_SOT_THT:TO-92_Inline" (at 90.17 98.425 0)
+    (property "Footprint" "Package_TO_SOT_THT:TO-92_Inline" (at 85.725 62.865 0)
       (effects (font (size 1.27 1.27) italic) (justify left) hide)
     )
-    (property "Datasheet" "https://www.onsemi.com/pub/Collateral/PN2222-D.PDF" (at 95.25 96.52 0)
+    (property "Datasheet" "https://www.onsemi.com/pub/Collateral/PN2222-D.PDF" (at 90.805 60.96 0)
       (effects (font (size 1.27 1.27)) (justify left) hide)
     )
@@
     )
   )
-  (symbol (lib_id "power:GND") (at 92.71 116.84 0) (unit 1)
-    (in_bom yes) (on_board yes) (dnp no) (fields_autoplaced)
-    (property "Reference" "#PWR046" (at 92.71 123.19 0)
-      (effects (font (size 1.27 1.27)) hide)
-    )
-    (property "Value" "GND" (at 92.71 121.92 0)
-      (effects (font (size 1.27 1.27)))
-    )
-    (property "Footprint" "" (at 92.71 116.84 0)
-      (effects (font (size 1.27 1.27)) hide)
-    )
-    (property "Datasheet" "" (at 92.71 116.84 0)
+  (symbol (lib_id "power:GND") (at 88.265 81.28 0) (unit 1)
+    (in_bom yes) (on_board yes) (dnp no) (fields_autoplaced)
+    (property "Reference" "#PWR046" (at 88.265 87.63 0)
+      (effects (font (size 1.27 1.27)) hide)
+    )
+    (property "Value" "GND" (at 88.265 86.36 0)
+      (effects (font (size 1.27 1.27)))
+    )
+    (property "Footprint" "" (at 88.265 81.28 0)
+      (effects (font (size 1.27 1.27)) hide)
+    )
+    (property "Datasheet" "" (at 88.265 81.28 0)
       (effects (font (size 1.27 1.27)) hide)
     )
@@
     )
   )
-  (symbol (lib_id "power:+5V") (at 92.71 83.82 0) (unit 1)
-    (in_bom yes) (on_board yes) (dnp no) (fields_autoplaced)
-    (property "Reference" "#PWR042" (at 92.71 87.63 0)
-      (effects (font (size 1.27 1.27)) hide)
-    )
-    (property "Value" "+5V" (at 92.71 79.375 0)
-      (effects (font (size 1.27 1.27)))
-    )
-    (property "Footprint" "" (at 92.71 83.82 0)
-      (effects (font (size 1.27 1.27)) hide)
-    )
-    (property "Datasheet" "" (at 92.71 83.82 0)
-      (effects (font (size 1.27 1.27)) hide)
-    )
+  (symbol (lib_id "power:+5V") (at 88.265 48.26 0) (unit 1)
+    (in_bom yes) (on_board yes) (dnp no) (fields_autoplaced)
+    (property "Reference" "#PWR042" (at 88.265 52.07 0)
+      (effects (font (size 1.27 1.27)) hide)
+    )
+    (property "Value" "+5V" (at 88.265 43.815 0)
+      (effects (font (size 1.27 1.27)))
+    )
+    (property "Footprint" "" (at 88.265 48.26 0)
+      (effects (font (size 1.27 1.27)) hide)
+    )
+    (property "Datasheet" "" (at 88.265 48.26 0)
+      (effects (font (size 1.27 1.27)) hide)
+    )

Commit message: discrete traces
Parts:
- renumbered C6 to C15, R9 to R10, R10 to R8, R8 to R9
Changed lines of the file:
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@@
   (symbol (lib_id "power:GND") (at 193.04 60.96 0) (unit 1)
     (in_bom yes) (on_board yes) (dnp no) (fields_autoplaced)
-    (property "Reference" "#PWR040" (at 193.04 67.31 0)
+    (property "Reference" "#PWR050" (at 193.04 67.31 0)
       (effects (font (size 1.27 1.27)) hide)
     )
@@
       (project "karca_v2"
         (path "/29cf4797-56f2-4f57-ae95-7df639362e3c/f3394041-f9fe-4d59-9036-d9e9f3f04b16"
-          (reference "#PWR040") (unit 1)
+          (reference "#PWR050") (unit 1)
         )
       )
@@
   (symbol (lib_id "Device:R_US") (at 232.41 64.77 0) (unit 1)
     (in_bom yes) (on_board yes) (dnp no) (fields_autoplaced)
-    (property "Reference" "R9" (at 234.95 63.5 0)
+    (property "Reference" "R10" (at 234.95 63.5 0)
       (effects (font (size 1.27 1.27)) (justify left))
     )
@@
       (project "karca_v2"
         (path "/29cf4797-56f2-4f57-ae95-7df639362e3c/f3394041-f9fe-4d59-9036-d9e9f3f04b16"
-          (reference "R9") (unit 1)
+          (reference "R10") (unit 1)
         )
       )
@@
   (symbol (lib_id "Device:R_US") (at 102.235 60.96 90) (unit 1)
     (in_bom yes) (on_board yes) (dnp no)
-    (property "Reference" "R10" (at 102.235 57.15 90)
+    (property "Reference" "R8" (at 102.235 57.15 90)
       (effects (font (size 1.27 1.27)))
     )
@@
       (project "karca_v2"
         (path "/29cf4797-56f2-4f57-ae95-7df639362e3c/f3394041-f9fe-4d59-9036-d9e9f3f04b16"
-          (reference "R10") (unit 1)
+          (reference "R8") (unit 1)
         )
       )
@@
   (symbol (lib_id "Device:C") (at 199.39 60.96 90) (unit 1)
     (in_bom yes) (on_board yes) (dnp no) (fields_autoplaced)
-    (property "Reference" "C6" (at 199.39 53.34 90)
+    (property "Reference" "C15" (at 199.39 53.34 90)
       (effects (font (size 1.27 1.27)))
     )
@@
       (project "karca_v2"
         (path "/29cf4797-56f2-4f57-ae95-7df639362e3c/f3394041-f9fe-4d59-9036-d9e9f3f04b16"
-          (reference "C6") (unit 1)
+          (reference "C15") (unit 1)
         )
       )
@@
   (symbol (lib_id "power:GND") (at 207.01 93.98 0) (unit 1)
     (in_bom yes) (on_board yes) (dnp no) (fields_autoplaced)
-    (property "Reference" "#PWR043" (at 207.01 100.33 0)
+    (property "Reference" "#PWR053" (at 207.01 100.33 0)
       (effects (font (size 1.27 1.27)) hide)
     )
@@
       (project "karca_v2"
         (path "/29cf4797-56f2-4f57-ae95-7df639362e3c/f3394041-f9fe-4d59-9036-d9e9f3f04b16"
-          (reference "#PWR043") (unit 1)
+          (reference "#PWR053") (unit 1)
         )
       )
@@
   (symbol (lib_id "power:+5V") (at 160.02 45.339 0) (unit 1)
     (in_bom yes) (on_board yes) (dnp no) (fields_autoplaced)
-    (property "Reference" "#PWR039" (at 160.02 49.149 0)
+    (property "Reference" "#PWR048" (at 160.02 49.149 0)
       (effects (font (size 1.27 1.27)) hide)
     )
@@
       (project "karca_v2"
         (path "/29cf4797-56f2-4f57-ae95-7df639362e3c/f3394041-f9fe-4d59-9036-d9e9f3f04b16"
-          (reference "#PWR039") (unit 1)
+          (reference "#PWR048") (unit 1)
         )
       )
@@
   (symbol (lib_id "Device:R_US") (at 215.9 64.77 0) (unit 1)
     (in_bom yes) (on_board yes) (dnp no)
-    (property "Reference" "R8" (at 210.82 63.5 0)
+    (property "Reference" "R9" (at 210.82 63.5 0)
       (effects (font (size 1.27 1.27)) (justify left))
     )
@@
       (project "karca_v2"
         (path "/29cf4797-56f2-4f57-ae95-7df639362e3c/f3394041-f9fe-4d59-9036-d9e9f3f04b16"
-          (reference "R8") (unit 1)
+          (reference "R9") (unit 1)
         )
       )
@@
   (symbol (lib_id "power:+5V") (at 208.28 60.96 0) (unit 1)
     (in_bom yes) (on_board yes) (dnp no)
-    (property "Reference" "#PWR041" (at 208.28 64.77 0)
+    (property "Reference" "#PWR051" (at 208.28 64.77 0)
       (effects (font (size 1.27 1.27)) hide)
     )
@@
       (project "karca_v2"
         (path "/29cf4797-56f2-4f57-ae95-7df639362e3c/f3394041-f9fe-4d59-9036-d9e9f3f04b16"
-          (reference "#PWR041") (unit 1)
+          (reference "#PWR051") (unit 1)
         )
       )
@@
   (symbol (lib_id "power:GND") (at 165.1 107.95 0) (unit 1)
     (in_bom yes) (on_board yes) (dnp no) (fields_autoplaced)
-    (property "Reference" "#PWR044" (at 165.1 114.3 0)
+    (property "Reference" "#PWR054" (at 165.1 114.3 0)
       (effects (font (size 1.27 1.27)) hide)
     )
@@
       (project "karca_v2"
         (path "/29cf4797-56f2-4f57-ae95-7df639362e3c/f3394041-f9fe-4d59-9036-d9e9f3f04b16"
-          (reference "#PWR044") (unit 1)
+          (reference "#PWR054") (unit 1)
         )
       )
@@
   (symbol (lib_id "power:GND") (at 88.265 81.28 0) (unit 1)
     (in_bom yes) (on_board yes) (dnp no) (fields_autoplaced)
-    (property "Reference" "#PWR046" (at 88.265 87.63 0)
+    (property "Reference" "#PWR052" (at 88.265 87.63 0)
       (effects (font (size 1.27 1.27)) hide)
     )
@@
       (project "karca_v2"
         (path "/29cf4797-56f2-4f57-ae95-7df639362e3c/f3394041-f9fe-4d59-9036-d9e9f3f04b16"
-          (reference "#PWR046") (unit 1)
+          (reference "#PWR052") (unit 1)
         )
       )
@@
   (symbol (lib_id "power:+5V") (at 88.265 48.26 0) (unit 1)
     (in_bom yes) (on_board yes) (dnp no) (fields_autoplaced)
-    (property "Reference" "#PWR042" (at 88.265 52.07 0)
+    (property "Reference" "#PWR049" (at 88.265 52.07 0)
       (effects (font (size 1.27 1.27)) hide)
     )
@@
       (project "karca_v2"
         (path "/29cf4797-56f2-4f57-ae95-7df639362e3c/f3394041-f9fe-4d59-9036-d9e9f3f04b16"
-          (reference "#PWR042") (unit 1)
+          (reference "#PWR049") (unit 1)
         )
       )
@@
   (symbol (lib_id "power:GND") (at 121.92 115.57 0) (unit 1)
     (in_bom yes) (on_board yes) (dnp no) (fields_autoplaced)
-    (property "Reference" "#PWR045" (at 121.92 121.92 0)
+    (property "Reference" "#PWR055" (at 121.92 121.92 0)
       (effects (font (size 1.27 1.27)) hide)
     )
@@
       (project "karca_v2"
         (path "/29cf4797-56f2-4f57-ae95-7df639362e3c/f3394041-f9fe-4d59-9036-d9e9f3f04b16"
-          (reference "#PWR045") (unit 1)
-        )
-      )
+          (reference "#PWR055") (unit 1)
+        )
+      )
