File: karca_v2/drivers.kicad_sch (KiCad schematic)
At the start: 13 parts, among them J10 Screw_Terminal_01x04, J11 Buzzer, J9 Screw_Terminal_01x10, Q4 AO3400A

Commit message: final production version
Parts:
- R16: MPN (none) -> C1493
- R17: MPN (none) -> C872846
Changed lines of the file:
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@@
+			)
+		)
+		(property "MPN" "C1493"
+			(at 140.335 157.48 0)
+			(effects
+				(font
+					(size 1.27 1.27)
+				)
+				(hide yes)
 			)
 		)
@@
 			(at 140.335 169.545 0)
 			(effects
+				(font
+					(size 1.27 1.27)
+				)
+				(hide yes)
+			)
+		)
+		(property "MPN" "C872846"
+			(at 140.335 169.545 0)
+			(effects
